File: bluetooth/bluetooth.sch (EAGLE design)
At the start: 6 parts

Commit message: Updated Boards for New Configuration
Bluetooth board has been rearranged to accommodate board slot-in
Motor Control Board flipped to be in the right spot
Parts:
- U$3, U$4: device RC Car:RESISTOR -> rc_car:RESISTOR

Commit message: Added breadboard board. This commit is going to production.
Parts:
- removed U$6: BT, RC Car:BT
- added U$5: HC-05, lib:HC-05
Connections:
- removed net 5V: POWER.POS, U$2.5V, U$6.VCC
- new net +5V: POWER.POS, U$2.5V, U$5.VCC
- net D03: now also U$5.TXD; no longer U$6.TXD
- net GND: now also U$1.GND, U$5.GND; no longer U$6.GND
- net RX: now also U$5.RXD; no longer U$6.RXD
