File: breadboard/breadboard.brd (EAGLE design)
At the start: 59.7 x 53.3 mm, 6 parts

Commit message: Added breadboard board. This commit is going to production.
Parts:
- removed POWER: CAP, RC Car:CAP
- removed U$1: ARDUINO-NANO-JUMPER-1, RC Car:ARDUINO-NANO-JUMPER-1
- removed U$3, U$4: RESISTOR, rc_car:RESISTOR
- U$2: value ARDUINO-NANO-JUMPER-2 -> ARDUINO-NANO-JUMPER-1; device RC Car:ARDUINO-NANO-JUMPER-2 -> RC Car:ARDUINO-NANO-JUMPER-1
- U$5: value HC-05 -> ARDUINO-NANO-JUMPER-2; device lib:HC-05 -> RC Car:ARDUINO-NANO-JUMPER-2
- moved U$2 45.7 mm to (30.5, 3.81), flipped to the bottom, turned to 0 degrees
- moved U$5 26.2 mm to (30.5, 49.5), flipped to the bottom, turned to 0 degrees
Connections:
- removed net +5V: POWER.POS, U$2.5V, U$5.VCC
- removed net D02: U$1.D2, U$3.POS
- removed net D03: U$1.D3, U$5.TXD
- removed net GND: POWER.NEG, U$1.GND, U$2.GND, U$4.NEG, U$5.GND
- removed net RX: U$3.NEG, U$4.POS, U$5.RXD
Routing:
- net GND: track 106.6 -> 0.00 mm, vias 2 -> 0
- net D03: track 96.8 -> 0.00 mm
- net RX: track 62.0 -> 0.00 mm
- net +5V: track 56.9 -> 0.00 mm
- net D02: track 20.5 -> 0.00 mm
Other:
- board text added: "A0"
- board text added: "A1"
- board text added: "A2"
- board text added: "A3"
- board text added: "A4"
- board text added: "A5"
- board text added: "A6"
- board text added: "A7"
- board text added: "D10"
- board text added: "D11"
- board text added: "D12"
- board text added: "D13"
- board text added: "D2"
- board text added: "D3"
- board text added: "D4"
- board text added: "D5"
- board text added: "D6"
- board text added: "D7"
- board text added: "D8"
- board text added: "D9"
- board text added: "RC CARS BREADBOARD V0.1"
- board text added: "REF"
- board text added: "RST"
- board text added: "RX0"
- board text added: "TX1"
- board text removed: "1k"
- board text removed: "2k"
- board text removed: "BLUETOOTH BOARD RC CARS V0.1"
