File: breadboard/breadboard.sch (EAGLE design)
At the start: 3 parts

Commit message: Added breadboard board. This commit is going to production.
Parts:
- removed U$1: ARDUINO-NANO-JUMPER-1, RC Car:ARDUINO-NANO-JUMPER-1
- removed U$7: ARDUINO-NANO-JUMPER-2, RC Car:ARDUINO-NANO-JUMPER-2
- added U$5: ARDUINO-NANO-JUMPER-2, RC Car:ARDUINO-NANO-JUMPER-2
- U$2: value L9110S -> ARDUINO-NANO-JUMPER-1; device RC Car:L9110S -> RC Car:ARDUINO-NANO-JUMPER-1
Connections:
- removed net D05: U$1.D05, U$2.A-1B
- removed net D06: U$1.D06, U$2.A-1A
- removed net GND: U$2.GND, U$7.GND
- removed net N$3: U$1.D11, U$2.B-1A
- removed net N$4: U$1.D10, U$2.B-2A
- removed net VIN: U$2.VCC, U$7.VIN
Changed lines of the file:
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@@
 </classes>
 <parts>
-<part name="U$1" library="RC Car" deviceset="ARDUINO-NANO-JUMPER-1" device=""/>
-<part name="U$2" library="RC Car" deviceset="L9110S" device=""/>
-<part name="U$7" library="RC Car" deviceset="ARDUINO-NANO-JUMPER-2" device=""/>
+<part name="U$2" library="RC Car" deviceset="ARDUINO-NANO-JUMPER-1" device=""/>
+<part name="U$5" library="RC Car" deviceset="ARDUINO-NANO-JUMPER-2" device=""/>
 </parts>
 <sheets>
@@
 </plain>
 <instances>
-<instance part="U$1" gate="G$1" x="71.12" y="30.48" smashed="yes"/>
-<instance part="U$2" gate="G$1" x="99.06" y="50.8" smashed="yes" rot="R270"/>
-<instance part="U$7" gate="G$1" x="154.94" y="68.58" smashed="yes" rot="R270"/>
+<instance part="U$2" gate="G$1" x="35.56" y="10.16" smashed="yes" rot="R270"/>
+<instance part="U$5" gate="G$1" x="-27.94" y="7.62" smashed="yes" rot="R270"/>
 </instances>
 <busses>
 </busses>
 <nets>
-<net name="D06" class="0">
-<segment>
-<pinref part="U$1" gate="G$1" pin="D06"/>
-<wire x1="71.12" y1="30.48" x2="71.12" y2="48.26" width="0.1524" layer="91"/>
-<pinref part="U$2" gate="G$1" pin="A-1A"/>
-<wire x1="71.12" y1="48.26" x2="93.98" y2="48.26" width="0.1524" layer="91"/>
-</segment>
-</net>
-<net name="D05" class="0">
-<segment>
-<pinref part="U$1" gate="G$1" pin="D05"/>
-<pinref part="U$2" gate="G$1" pin="A-1B"/>
-<wire x1="73.66" y1="30.48" x2="73.66" y2="45.72" width="0.1524" layer="91"/>
-<wire x1="73.66" y1="45.72" x2="93.98" y2="45.72" width="0.1524" layer="91"/>
-</segment>
-</net>
-<net name="GND" class="0">
-<segment>
-<pinref part="U$2" gate="G$1" pin="GND"/>
-<wire x1="93.98" y1="53.34" x2="154.94" y2="53.34" width="0.1524" layer="91"/>
-<pinref part="U$7" gate="G$1" pin="GND"/>
-</segment>
-</net>
-<net name="VIN" class="0">
-<segment>
-<pinref part="U$7" gate="G$1" pin="VIN"/>
-<pinref part="U$2" gate="G$1" pin="VCC"/>
-<wire x1="154.94" y1="50.8" x2="93.98" y2="50.8" width="0.1524" layer="91"/>
-</segment>
-</net>
-<net name="N$4" class="0">
-<segment>
-<pinref part="U$1" gate="G$1" pin="D10"/>
-<wire x1="60.96" y1="30.48" x2="60.96" y2="55.88" width="0.1524" layer="91"/>
-<wire x1="60.96" y1="55.88" x2="93.98" y2="55.88" width="0.1524" layer="91"/>
-<pinref part="U$2" gate="G$1" pin="B-2A"/>
-</segment>
-</net>
-<net name="N$3" class="0">
-<segment>
-<pinref part="U$2" gate="G$1" pin="B-1A"/>
-<wire x1="93.98" y1="58.42" x2="58.42" y2="58.42" width="0.1524" layer="91"/>
-<wire x1="58.42" y1="58.42" x2="58.42" y2="30.48" width="0.1524" layer="91"/>
-<pinref part="U$1" gate="G$1" pin="D11"/>
-</segment>
-</net>
 </nets>
 </sheet>
